Commit message: add dummy inertia for root links st. rbdl find the root link

File: models/hyq.urdf (robot description, URDF)
Before this commit: robot hyq, 19 links, 18 joints
Links:
- link base_link: mass None -> 0.000001

File: models/nao.urdf (robot description, URDF)
Before this commit: robot nao, 33 links, 32 joints
Links:
- link base_link: mass None -> 0.000001

File: models/romeo.urdf (robot description, URDF)
Before this commit: robot romeoH37V1, 58 links, 57 joints
Links:
- link base_link: mass None -> 0.000001
