Commit message: done

File: models/lwr.urdf (robot description, URDF)
Before this commit: robot kuka-lwr2, 9 links, 8 joints
Links:
- link world_link: mass 50.0 -> None

Commit message: model: correct LWR

File: models/lwr.urdf (robot description, URDF)
Before this commit: robot kuka-lwr2, 9 links, 8 joints
Links:
- removed link world_link
- added link base_link; collision box size=0.5 0.5 0.05; visual box size=0.5 0.5 0.05
Joints:
- joint world_lwr_arm_base_joint: parent world_link -> base_link
